File: PCB/RoomUnit_MQTT_PCB/RoomUnit_MQTT_PCB.kicad_pcb (KiCad board)
At the start: 2 copper layers, 40 x 60 mm, 26 parts, among them J1 Conn_01x08_Socket, Q1 MMBTA06, U1 LMV393, U2 MOUDLE-SEEEDUINO-XIAO-ESP32C3, U3 L78L24_SOT89

Commit message: pcb progress
Parts:
- removed R4, R7: 18k, Resistor_SMD:R_0805_2012Metric_Pad1.20x1.40mm_HandSolder
- removed U2: MOUDLE-SEEEDUINO-XIAO-ESP32C3, RF_Module:MCU_Seeed_ESP32C3
- added J2: Conn_01x07_Socket, Project_Library:XIAO_ESP32-C3_Custom_Connector, F.Cu at (158.0, 98.0)
- added U4: ~, Project_Library:RoomUnit_Connector_5mm, F.Cu at (152.3, 42.7)
- J1: value Conn_01x08_Socket -> Conn_01x07_Socket; footprint Connector_Samtec_HPM_THT:Samtec_HPM-08-01-x-S_Straight_1x08_Pitch5.08mm -> Project_Library:XIAO_ESP32-C3_Custom_Connector
- moved J1 59.1 mm to (176.3, 98.0), turned to 180 degrees
- moved D2 57.5 mm to (165.5, 55.0), turned to 180 degrees
- moved C2 55.3 mm to (161.5, 55.0), turned to 180 degrees
- moved R2 45.8 mm to (162.5, 68.0)
- moved R3 45.4 mm to (162.5, 70.0)
- moved C1 45.2 mm to (169.5, 66.0), turned to 180 degrees
- moved R6 42.4 mm to (176.5, 72.0)
- moved R9 42.0 mm to (165.5, 52.7), turned to 180 degrees
- moved R5 41.0 mm to (176.5, 70.0), turned to 180 degrees
- moved R8 36.4 mm to (176.5, 68.0), turned to 180 degrees
- moved L1 20.2 mm to (175.5, 57.5), turned to -90 degrees
- moved R1 19.2 mm to (162.5, 74.0), turned to 180 degrees
- moved D1 15.8 mm to (161.5, 58.5)
- moved R14 13.6 mm to (162.5, 72.0), turned to 180 degrees
- moved C4 8.50 mm to (163.0, 50.0)
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Connections:
- J1 pad 1: GND -> Net-(J1-Pin_1)
- J1 pad 2: +24V -> Net-(J1-Pin_2)
- J1 pad 3: MPS -> Net-(J1-Pin_3)
- J1 pad 4: GND -> unconnected-(J1-Pin_4-Pad4)
- J1 pad 6: AO1 -> unconnected-(J1-Pin_6-Pad6)
- J1 pad 7: AO2 -> Net-(J1-Pin_7)
- R10 pad 2: Net-(U2-PA02_A0_D0) -> Net-(J1-Pin_1)
- R11 pad 2: Net-(U2-PA4_A1_D1) -> Net-(J1-Pin_2)
- R12 pad 2: Net-(U2-PA10_A2_D2) -> Net-(J1-Pin_3)
- R13 pad 2: Net-(U2-PB08_A6_D6_TX) -> Net-(J1-Pin_7)
Routing:
- net +5V: track 0.00 -> 70.9 mm, vias 0 -> 1
- net +3V3: track 0.00 -> 58.3 mm, vias 0 -> 1
- net AO1: track 0.00 -> 57.2 mm
- net AO2: track 0.00 -> 50.4 mm
- net AO3: track 0.00 -> 44.2 mm
- net UART_TX: track 0.00 -> 21.7 mm, vias 0 -> 2
- net Net-(J2-Pin_7): track 0.00 -> 20.3 mm, vias 0 -> 1
- net MPS: track 0.00 -> 16.6 mm
- net UART_RX: track 0.00 -> 13.1 mm
- net Net-(U1A-+): track 0.00 -> 12.8 mm
- net Net-(U1A--): track 0.00 -> 11.8 mm
- net +24V: track 0.00 -> 11.7 mm
- net Net-(D2-K): track 0.00 -> 9.06 mm
- net Net-(Q1-B): track 0.00 -> 7.53 mm
- net Net-(Q1-C): track 0.00 -> 4.56 mm
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- added copper zone on B.Cu, net GND
- added copper zone on F.Cu, net GND
Other:
- board size 40 x 60 mm -> 34.3 x 60 mm
